File: GPS-SIM5320-3G-MICROMOD-Male/GPS-SIM5320-3G-MICROMOD-Male.brd (EAGLE design)
At the start: 37.3 x 42.1 mm, 31 parts, among them IC1 74VHCT125PW, Q2 bss138, U1 SIM5320, X1 uFL, X2 uFL

Commit message: Add files via upload
Parts:
- R2: value 10K -> 10
Other:
- board text added: "GPS_ANT"
- board text added: "GPS_SELECT"
- board text added: "GSM_ANT"
- board text added: "SIM_CARD"
