File: GPS-SIM5320-3G-MICROMOD-Male/GPS-SIM5320-3G-MICROMOD-Male.sch (EAGLE design)
At the start: 31 parts, among them IC1 74VHCT125PW, Q2 bss138, U1 SIM5320, X1 uFL, X2 uFL

Commit message: Add files via upload
Parts:
- R2: value 10K -> 10
Changed lines of the file:
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@@
 <part name="D5" library="microbuilder" deviceset="DIODE" device="SOD-323" value="1N4148"/>
 <part name="D7" library="microbuilder" deviceset="DIODE" device="SOD-323" value="1N4148"/>
-<part name="R2" library="microbuilder" deviceset="RESISTOR" device="0805_NOOUTLINE" value="10K"/>
+<part name="R2" library="microbuilder" deviceset="RESISTOR" device="0805_NOOUTLINE" value="10"/>
 <part name="MMM1" library="Micromod_4222_Male_NoDim" deviceset="MICROMOD_4222_MALE" device=""/>
 <part name="VIO" library="microbuilder" deviceset="2.8V" device=""/>
@@
 <instance part="R2" gate="G$1" x="309.88" y="213.36" smashed="yes" rot="R90">
 <attribute name="NAME" x="307.34" y="213.36" size="1.27" layer="95" font="vector" rot="R90" align="center"/>
-<attribute name="VALUE" x="309.88" y="210.82" size="1.016" layer="96" font="vector" ratio="15" rot="R90" align="center"/>
+<attribute name="VALUE" x="309.88" y="213.36" size="1.016" layer="96" font="vector" ratio="15" rot="R90" align="center"/>
 </instance>
 <instance part="MMM1" gate="G$1" x="132.08" y="63.5" smashed="yes">
